File: PCB/PCB.kicad_pcb (KiCad board)
At the start: 2 copper layers, 39 parts, among them J1 Conn_01x07_Pin, J2 Conn_01x07_Pin, J3 Conn_01x04_Pin, J4 USB_C_Receptacle_USB2.0_14P, SW1 SW_Push, SW2 SW_Push, SW3 SW_Push, U1 RP2040, U2 MCP1700, U3 W25Q128JVS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

Commit message: potato
Parts:
- removed SW1: SW_Push, Taranium-libs:C720477
- added J5: Conn_01x03_Pin, Connector_PinSocket_2.54mm:PinSocket_1x03_P2.54mm_Vertical, F.Cu at (169.4, 58.5)
- C1, C8: value 0.1uf -> 1uf
- J3: value Conn_01x04_Pin -> Conn_01x06_Pin; footprint Connector_PinSocket_2.54mm:PinSocket_1x04_P2.54mm_Vertical -> Connector_PinSocket_2.54mm:PinSocket_1x06_P2.54mm_Vertical
- U2: footprint Package_SON:Winbond_USON-8-1EP_3x2mm_P0.5mm_EP0.2x1.6mm -> Package_TO_SOT_SMD:SOT-23_Handsoldering
- moved SW3 73.4 mm to (169.8, 65.6), turned to -90 degrees
- moved U2 67.9 mm to (158.3, 74.0), turned to -90 degrees
- moved U4 66.6 mm to (163.5, 73.2), turned to 90 degrees
- moved D1 66.5 mm to (168.9, 74.4), turned to -90 degrees
- moved C13 58.8 mm to (142.4, 64.4)
- moved C16 56.5 mm to (167.8, 68.6), turned to -90 degrees
- moved C1 56.5 mm to (142.3, 70.2), turned to -90 degrees
- moved C14 54.4 mm to (138.6, 68.5), turned to 90 degrees
- moved C15 54.1 mm to (165.9, 73.1), turned to 90 degrees
- moved Y1 52.7 mm to (141.5, 66.6)
- moved C11 51.5 mm to (161.0, 74.2), turned to 90 degrees
- moved J4 49.9 mm to (163.6, 79.4), turned to 90 degrees
- moved C12 47.0 mm to (155.7, 73.9), turned to -90 degrees
- moved C7 45.9 mm to (154.0, 69.6)
- moved C6 44.9 mm to (152.2, 64.5), turned to 90 degrees
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Connections:
- C12 pad 1: Net-(U2-VO) -> +3V3
- J1 pad 1: VBUS -> GPIO0
- J1 pad 2: unconnected-(J1-Pin_2-Pad2) -> GPIO1
- J1 pad 3: unconnected-(J1-Pin_3-Pad3) -> GPIO2
- J1 pad 4: unconnected-(J1-Pin_4-Pad4) -> GPIO3
- J1 pad 5: unconnected-(J1-Pin_5-Pad5) -> GPIO4
- J1 pad 6: unconnected-(J1-Pin_6-Pad6) -> GPIO5
- J1 pad 7: unconnected-(J1-Pin_7-Pad7) -> GPIO6
- J1 pad 8: unconnected-(J1-Pin_8-Pad8) -> GPIO7
- J2 pad 2: unconnected-(J2-Pin_2-Pad2) -> GND
- J2 pad 3: unconnected-(J2-Pin_3-Pad3) -> GPIO28
- J2 pad 4: unconnected-(J2-Pin_4-Pad4) -> GPIO27
- J2 pad 5: unconnected-(J2-Pin_5-Pad5) -> GPIO26
- J2 pad 6: unconnected-(J2-Pin_6-Pad6) -> GPIO25
- J2 pad 7: unconnected-(J2-Pin_7-Pad7) -> GPIO24
- J2 pad 8: unconnected-(J2-Pin_8-Pad8) -> GPIO23
- J3 pad 1: unconnected-(J3-Pin_1-Pad1) -> GPIO18
- J3 pad 2: unconnected-(J3-Pin_2-Pad2) -> GPIO17
- J3 pad 3: unconnected-(J3-Pin_3-Pad3) -> GND
- J3 pad 4: unconnected-(J3-Pin_4-Pad4) -> GPIO10
- U2 pad 2: Net-(U2-VO) -> +3V3
Routing:
- net +3V3: track 0.00 -> 98.4 mm, vias 0 -> 10
- net GND: track 0.00 -> 66.7 mm, vias 0 -> 62
- net VBUS: track 0.00 -> 41.6 mm, vias 0 -> 1
- net SPI_SS: track 0.00 -> 20.1 mm
- net GPIO23: track 0.00 -> 19.1 mm
- net GPIO7: track 0.00 -> 18.3 mm
- net +1V1: track 0.00 -> 17.9 mm, vias 0 -> 3
- net GPIO24: track 0.00 -> 17.0 mm
- net Net-(D1-A): track 0.00 -> 16.9 mm
- net GPIO6: track 0.00 -> 16.3 mm
- net GPIO25: track 0.00 -> 15.0 mm
- net GPIO5: track 0.00 -> 14.3 mm
- net GPIO9: track 0.00 -> 14.3 mm
- net GPIO8: track 0.00 -> 14.1 mm
- net GPIO10: track 0.00 -> 13.9 mm, vias 0 -> 1
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- added copper zone on B.Cu, net GND
- added copper zone on F.Cu, net GND
Other:
- board outline added: 39.1 x 26.9 mm

Commit message: commit arson
Parts:
- BOOT: renamed from SW3; value SW_Push -> BOOT
- J1, J2, J3, J5: moved to B.Cu
- RESET: renamed from SW2; value SW_Push -> RESET
- moved R8 4.18 mm to (161.0, 59.1), turned to -45 degrees
- moved C16 4.17 mm to (165.6, 65.0)
- moved C13 1.90 mm to (144.2, 65.2), turned to -90 degrees
- moved D2 0.86 mm to (169.5, 69.9)
- moved R4 0.28 mm to (167.0, 70.3)
- moved RESET 0.10 mm to (138.1, 74.1)
- turned J1 to 90 degrees
- turned J2 to 90 degrees
- turned J3 to 0 degrees
- turned J5 to 90 degrees
Connections:
- J3 pad 4: GPIO10 -> RUN
Routing:
- net GPIO10: track 13.9 -> 0.00 mm, vias 1 -> 0
- net RUN: track 7.74 -> 12.9 mm
- net Net-(BOOT1-Pad2): track 5.62 -> 9.99 mm
- net SPI_SS: track 20.1 -> 21.9 mm
- net GND: track 66.7 -> 67.7 mm, vias 62 -> 80
- net +1V1: track 17.9 -> 18.7 mm
- net +3V3: track 98.4 -> 97.8 mm
Other:
- board text added: "00"
- board text added: "01"
- board text added: "02"
- board text added: "03"
- board text added: "04"
- board text added: "05"
- board text added: "06"
- board text added: "07"
- board text added: "08"
- board text added: "09"
- board text added: "17"
- board text added: "18"
- board text added: "23"
- board text added: "24"
- board text added: "25"
- board text added: "26"
- board text added: "27"
- board text added: "28"
- board text added: "3V3"
- board text added: "GND"
- board text added: "RUN"
- board text added: "VBUS"
