File: PCB/PCB.kicad_pcb (KiCad board)
At the start: 2 copper layers, 39.1 x 26.9 mm, 39 parts, among them J1 Conn_01x07_Pin, J2 Conn_01x07_Pin, J3 Conn_01x06_Pin, J4 USB_C_Receptacle_USB2.0_14P, J5 Conn_01x03_Pin, U1 RP2040, U2 MCP1700, U3 W25Q128JVS, U4 USBLC6-2SC6, Y1 12MHz

Commit message: production and stuff
Parts:
- J1, J2: footprint Connector_PinSocket_2.54mm:PinSocket_1x08_P2.54mm_Vertical -> Connector_PinHeader_2.54mm:PinHeader_1x08_P2.54mm_Vertical
- J3: footprint Connector_PinSocket_2.54mm:PinSocket_1x06_P2.54mm_Vertical -> Connector_PinHeader_2.54mm:PinHeader_1x06_P2.54mm_Vertical
- J5: footprint Connector_PinSocket_2.54mm:PinSocket_1x03_P2.54mm_Vertical -> Connector_PinHeader_2.54mm:PinHeader_1x03_P2.54mm_Vertical
