File: PCB/PCB.kicad_pcb (KiCad board)
At the start: 2 copper layers, 39.1 x 26.9 mm, 39 parts, among them J1 Conn_01x07_Pin, J2 Conn_01x07_Pin, J3 Conn_01x06_Pin, J4 USB_C_Receptacle_USB2.0_14P, J5 Conn_01x03_Pin, U1 RP2040, U2 MCP1700, U3 W25Q128JVS, U4 USBLC6-2SC6, Y1 12MHz

Commit message: potato
Parts:
- J1, J2: value Conn_01x07_Pin -> Conn_01x08_Pin; footprint Connector_PinHeader_2.54mm:PinHeader_1x08_P2.54mm_Vertical -> Connector_PinSocket_2.54mm:PinSocket_1x08_P2.54mm_Vertical
- J3: footprint Connector_PinHeader_2.54mm:PinHeader_1x06_P2.54mm_Vertical -> Connector_PinSocket_2.54mm:PinSocket_1x06_P2.54mm_Vertical
- J5: footprint Connector_PinHeader_2.54mm:PinHeader_1x03_P2.54mm_Vertical -> Connector_PinSocket_2.54mm:PinSocket_1x03_P2.54mm_Vertical
- renumbered BOOT to BOOT1, RESET to RESET1

Commit message: potato
Parts:
- J1, J2: footprint Connector_PinSocket_2.54mm:PinSocket_1x08_P2.54mm_Vertical -> Connector_PinHeader_2.54mm:PinHeader_1x08_P2.54mm_Vertical
- J3: footprint Connector_PinSocket_2.54mm:PinSocket_1x06_P2.54mm_Vertical -> Connector_PinHeader_2.54mm:PinHeader_1x06_P2.54mm_Vertical
- J5: footprint Connector_PinSocket_2.54mm:PinSocket_1x03_P2.54mm_Vertical -> Connector_PinHeader_2.54mm:PinHeader_1x03_P2.54mm_Vertical
- moved J5 0.79 mm to (170.2, 58.5)
Routing:
- net +3V3: track 98.3 -> 97.2 mm

Commit message: potato
Parts:
- J1, J2: footprint Connector_PinHeader_2.54mm:PinHeader_1x08_P2.54mm_Vertical -> Connector_PinSocket_2.54mm:PinSocket_1x08_P2.54mm_Vertical
- J3: footprint Connector_PinHeader_2.54mm:PinHeader_1x06_P2.54mm_Vertical -> Connector_PinSocket_2.54mm:PinSocket_1x06_P2.54mm_Vertical
- J5: footprint Connector_PinHeader_2.54mm:PinHeader_1x03_P2.54mm_Vertical -> Connector_PinSocket_2.54mm:PinSocket_1x03_P2.54mm_Vertical
- R4: value 2.2 -> 2.2k
- R5, R6: value 22k -> 5.1k
