File: PCB/PCB.kicad_sch (KiCad schematic)
At the start: 6 parts, among them J1 Conn_01x07_Pin, J2 Conn_01x07_Pin, J3 Conn_01x04_Pin, U1 RP2040

Commit message: im gonna meta post nimit
Parts:
- added C10, C11, C12, C2, C3, C4, C5, C6, C7, C8, C9: C_Small, symbol Device:C_Small
- added D2: LED, symbol Device:LED
- added J4: USB_C_Receptacle_USB2.0_14P, symbol Connector:USB_C_Receptacle_USB2.0_14P
- added R1, R2, R3, R4: R_Small, symbol Device:R_Small
- added SW1, SW2: SW_Push, symbol Switch:SW_Push
- added U2: NCP1117-3.3_SOT223, Package_TO_SOT_SMD:SOT-223-3_TabPin2, symbol Regulator_Linear:NCP1117-3.3_SOT223
- added U3: W25Q128JVS, Package_SO:SOIC-8_5.3x5.3mm_P1.27mm, symbol Memory_Flash:W25Q128JVS
- added Y1: Crystal_GND23_Small, symbol Device:Crystal_GND23_Small
Connections:
- net at U1.26 (RUN): now also R3.1, SW2.2
- net at U1.46 (USB_DM): now also R2.2
- net at U1.47 (USB_DP): now also R1.2
- net GND: now reaches U1.57 (GND)
- net GND: now also C1.2, C10.2, C11.2, C12.2, C2.2, C3.2, C4.2, C5.2, C6.2, C7.2, C8.2, C9.2, D2.1 (K), J4.A1 (GND), J4.A12 (GND), J4.B1 (GND), J4.B12 (GND), J4.S1 (SHIELD), SW2.1, U2.1 (GND), U3.4 (GND)
- net +3V3: now reaches C1.1
- net +3V3: now also C2.1, C3.1, C4.1, C5.1, C6.1, C7.1, R3.2, R4.2
- new net: D2.2 (A), R4.1
- new net: C11.1, U2.3 (VI)
- new net: J4.A4 (VBUS), J4.A9 (VBUS), J4.B4 (VBUS), J4.B9 (VBUS)
- new net: J4.A6 (D+), J4.B6 (D+)
- new net: J4.A7 (D-), J4.B7 (D-)
- new net: C12.1, U2.2 (VO)
- new net +1V1: C10.1, C8.1, C9.1
Other:
- moved on the sheet: C1, J1, J2, J3, U1

Commit message: potato
Parts:
- removed Y1: Crystal_GND23_Small, symbol Device:Crystal_GND23_Small
- added C13, C14: C_Small, symbol Device:C_Small
- added R5, R6, R7, R8, R9: R_Small, symbol Device:R_Small
- added SW3: SW_Push, symbol Switch:SW_Push
- added Y1: Crystal_GND24, symbol Device:Crystal_GND24
Connections:
- net +3V3: now also U3.8 (VCC), R9.1
- net GND: now also C13.1, C14.1, R5.1, R6.1, SW3.1, Y1.2, Y1.4
- net at C11.1, U2.3 (VI): now also J4.A4 (VBUS), J4.A9 (VBUS), J4.B4 (VBUS), J4.B9 (VBUS)
- net at J4.A5 (CC1): now also R5.2
- net at J4.B5 (CC2): now also R6.2
- net at U3.1 (~{CS}): now also R8.1, R9.2
- new net: C14.2, R7.2, Y1.1
- new net: C13.2, Y1.3
- new net: R8.2, SW3.2

Commit message: bleh
Parts:
- added C15, C16: C_Small, symbol Device:C_Small
- added U4: USBLC6-2SC6, Package_TO_SOT_SMD:SOT-23-6, symbol Power_Protection:USBLC6-2SC6
Connections:
- net +1V1: now also U1.23 (DVDD), U1.45 (VREG_VOUT), U1.50 (DVDD)
- net +3V3: now also U1.1 (IOVDD), U1.10 (IOVDD), U1.22 (IOVDD), U1.33 (IOVDD), U1.42 (IOVDD), U1.43 (ADC_AVDD), U1.44 (VREG_IN), U1.48 (USB_VDD), U1.49 (IOVDD), C16.1
- net GND: now also U1.19 (TESTEN), C15.2, C16.2, U4.2 (GND)
- net XIN: now reaches C13.2, Y1.3
- net XIN: now also U1.20 (XIN)
- net VBUS: now reaches J1.1 (Pin_1)
- net VBUS: now also D1.1 (K), C15.1, U4.5 (VBUS)
- net SPI_SS: now reaches R8.1, R9.2, U3.1 (~{CS})
- net SPI_SS: now also U1.56 (QSPI_SS)
- net GPIO8: now reaches U1.11 (GPIO8)
- net GPIO9: now reaches U1.12 (GPIO9)
- net GPIO10: now reaches U1.13 (GPIO10)
- net GPIO11: now reaches U1.14 (GPIO11)
- net GPIO12: now reaches U1.15 (GPIO12)
- net GPIO13: now reaches U1.16 (GPIO13)
- net GPIO14: now reaches U1.17 (GPIO14)
- net GPIO15: now reaches U1.18 (GPIO15)
- net GPIO0: now reaches U1.2 (GPIO0)
- net XOUT: now reaches U1.21 (XOUT)
- net XOUT: now also R7.1
- net GPIO16: now reaches U1.27 (GPIO16)
- net GPIO17: now reaches U1.28 (GPIO17)
- net GPIO18: now reaches U1.29 (GPIO18)
- net GPIO1: now reaches U1.3 (GPIO1)
- net GPIO19: now reaches U1.30 (GPIO19)
- net GPIO20: now reaches U1.31 (GPIO20)
- net GPIO21: now reaches U1.32 (GPIO21)
- net GPIO22: now reaches U1.34 (GPIO22)
- net GPIO23: now reaches U1.35 (GPIO23)
- net GPIO24: now reaches U1.36 (GPIO24)
- net GPIO25: now reaches U1.37 (GPIO25)
- net GPIO26: now reaches U1.38 (GPIO26_ADC0)
- net GPIO27: now reaches U1.39 (GPIO27_ADC1)
- net GPIO2: now reaches U1.4 (GPIO2)
- net GPIO28: now reaches U1.40 (GPIO28_ADC2)
- net GPIO29: now reaches U1.41 (GPIO29_ADC3)
- net GPIO3: now reaches U1.5 (GPIO3)
- net SPI_SD3: now reaches U1.51 (QSPI_SD3)
- net SPI_SD3: now also U3.7 (~{HOLD}/~{RESET}/IO_{3})
- net SPI_SCLK: now reaches U1.52 (QSPI_SCLK)
- net SPI_SCLK: now also U3.6 (CLK)
- net SPI_SD0: now reaches U1.53 (QSPI_SD0)
- net SPI_SD0: now also U3.5 (DI/IO_{0})
- net SPI_SD2: now reaches U1.54 (QSPI_SD2)
- net SPI_SD2: now also U3.3 (~{WP}/IO_{2})
- net SPI_SD1: now reaches U1.55 (QSPI_SD1)
- net SPI_SD1: now also U3.2 (DO/IO_{1})
- net GPIO4: now reaches U1.6 (GPIO4)
- net GPIO5: now reaches U1.7 (GPIO5)
- net GPIO6: now reaches U1.8 (GPIO6)
- net GPIO7: now reaches U1.9 (GPIO7)
- net at C11.1, J4.A4 (VBUS), J4.A9 (VBUS)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: now also D1.2 (A)
- net at J4.A6 (D+), J4.B6 (D+): now also U4.3 (I/O2)
- net at J4.A7 (D-), J4.B7 (D-): now also U4.1 (I/O1)
- net DP: now reaches R1.1
- net DP: now also U4.4 (I/O2)
- net DM: now reaches R2.1
- net DM: now also U4.6 (I/O1)
Other:
- moved on the sheet: D1

Commit message: havent commited in a while
Parts:
- C1, C10, C15, C16, C2, C3, C4, C5, C6, C7, C8, C9: value C_Small -> 0.1uf; footprint (none) -> Capacitor_SMD:C_0402_1005Metric_Pad0.74x0.62mm_HandSolder
- C11, C12: value C_Small -> 10uf; footprint (none) -> Capacitor_SMD:C_0603_1608Metric_Pad1.08x0.95mm_HandSolder
- C13, C14: value C_Small -> 15pf; footprint (none) -> Capacitor_SMD:C_0402_1005Metric_Pad0.74x0.62mm_HandSolder
- D1: value D_Small -> C48192; footprint (none) -> Diode_SMD:D_SOD-323_HandSoldering
- D2: footprint (none) -> LED_SMD:LED_0805_2012Metric_Pad1.15x1.40mm_HandSolder
- J1, J2: footprint (none) -> Connector_PinSocket_2.54mm:PinSocket_1x08_P2.54mm_Vertical; symbol Connector:Conn_01x07_Pin -> Connector:Conn_01x08_Pin
- J3: footprint (none) -> Connector_PinSocket_2.54mm:PinSocket_1x04_P2.54mm_Vertical
- J4: footprint (none) -> Taranium-libs:USB-C-SMD_20P-P0.50-L6.5-W8.9
- R1, R2: value R_Small -> 27; footprint (none) -> Resistor_SMD:R_0402_1005Metric_Pad0.72x0.64mm_HandSolder
- R3, R9: value R_Small -> 10k; footprint (none) -> Resistor_SMD:R_0402_1005Metric_Pad0.72x0.64mm_HandSolder
- R4: value R_Small -> 2.2; footprint (none) -> Resistor_SMD:R_0402_1005Metric_Pad0.72x0.64mm_HandSolder
- R5, R6: value R_Small -> 22k; footprint (none) -> Resistor_SMD:R_0402_1005Metric_Pad0.72x0.64mm_HandSolder
- R7, R8: value R_Small -> 1k; footprint (none) -> Resistor_SMD:R_0402_1005Metric_Pad0.72x0.64mm_HandSolder
- SW1, SW2, SW3: footprint (none) -> Taranium-libs:C720477
- U2: value NCP1117-3.3_SOT223 -> MCP1700; footprint Package_TO_SOT_SMD:SOT-223-3_TabPin2 -> Package_SON:Winbond_USON-8-1EP_3x2mm_P0.5mm_EP0.2x1.6mm
- Y1: value Crystal_GND24 -> 12MHz; footprint (none) -> Taranium-libs:CRYSTAL-SMD_4P-L3.2-W2.5-BL
Connections:
- net VBUS: now also J2.1 (Pin_1)
- net RUN: now reaches R3.1, SW2.2, U1.26 (RUN)
Other:
- moved on the sheet: SW2

Commit message: potato
Parts:
- removed SW1: SW_Push, Taranium-libs:C720477, symbol Switch:SW_Push
- added J5: Conn_01x03_Pin, Connector_PinSocket_2.54mm:PinSocket_1x03_P2.54mm_Vertical, symbol Connector:Conn_01x03_Pin
- C1, C8: value 0.1uf -> 1uf
- J3: value Conn_01x04_Pin -> Conn_01x06_Pin; footprint Connector_PinSocket_2.54mm:PinSocket_1x04_P2.54mm_Vertical -> Connector_PinSocket_2.54mm:PinSocket_1x06_P2.54mm_Vertical; symbol Connector:Conn_01x04_Pin -> Connector:Conn_01x06_Pin
- U2: footprint Package_SON:Winbond_USON-8-1EP_3x2mm_P0.5mm_EP0.2x1.6mm -> Package_TO_SOT_SMD:SOT-23_Handsoldering
Connections:
- net +3V3: now also C12.1, U2.2 (VO), J5.3 (Pin_3)
- net GND: now also J2.2 (Pin_2), J3.3 (Pin_3), J5.2 (Pin_2)
- net GPIO0: now also J1.1 (Pin_1)
- net GPIO1: now also J1.2 (Pin_2)
- net GPIO10: now also J3.4 (Pin_4)
- net GPIO17: now also J3.2 (Pin_2)
- net GPIO18: now also J3.1 (Pin_1)
- net GPIO2: now also J1.3 (Pin_3)
- net GPIO23: now also J2.8 (Pin_8)
- net GPIO24: now also J2.7 (Pin_7)
- net GPIO25: now also J2.6 (Pin_6)
- net GPIO26: now also J2.5 (Pin_5)
- net GPIO27: now also J2.4 (Pin_4)
- net GPIO28: now also J2.3 (Pin_3)
- net GPIO3: now also J1.4 (Pin_4)
- net GPIO4: now also J1.5 (Pin_5)
- net GPIO5: now also J1.6 (Pin_6)
- net GPIO6: now also J1.7 (Pin_7)
- net GPIO7: now also J1.8 (Pin_8)
- net GPIO8: now also J3.6 (Pin_6)
- net GPIO9: now also J3.5 (Pin_5)
- net VBUS: now also J5.1 (Pin_1); no longer J1.1 (Pin_1)

Commit message: commit arson
Parts:
- BOOT: renamed from SW3; value SW_Push -> BOOT
- RESET: renamed from SW2; value SW_Push -> RESET
Connections:
- net GPIO10: no longer J3.4 (Pin_4)
- net RUN: now also J3.4 (Pin_4)
Changed lines of the file:
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@@
 		)
 	)
+	(global_label "RUN"
+		(shape input)
+		(at 156.21 187.96 90)
+		(fields_autoplaced yes)
+		(effects
+			(font
+				(size 1.27 1.27)
+			)
+			(justify left)
+		)
+		(property "Intersheetrefs" "${INTERSHEET_REFS}"
+			(at 156.21 181.0438 90)
+			(effects
+				(font
+					(size 1.27 1.27)
+				)
+				(justify left)
+				(hide yes)
+			)
+		)
+	)
 	(global_label "GPIO28"
 		(shape input)
@@
 		)
 	)
-	(global_label "GPIO10"
-		(shape input)
-		(at 156.21 187.96 90)
-		(fields_autoplaced yes)
-		(effects
-			(font
-				(size 1.27 1.27)
-			)
-			(justify left)
-		)
-		(property "Intersheetrefs" "${INTERSHEET_REFS}"
-			(at 156.21 178.0805 90)
-			(effects
-				(font
-					(size 1.27 1.27)
-				)
-				(justify left)
-				(hide yes)
-			)
-		)
-	)
 	(global_label "GPIO14"
 		(shape input)
@@
 		(dnp no)
 		(fields_autoplaced yes)
-		(property "Reference" "SW3"
+		(property "Reference" "BOOT"
 			(at 154.94 52.07 0)
 			(effects
@@
 			)
 		)
-		(property "Value" "SW_Push"
+		(property "Value" "BOOT"
 			(at 154.94 54.61 0)
 			(effects
@@
 			(project "PCB"
 				(path "/7d2cf6c2-cd4f-44e4-8c0c-48fa8c8e68c1"
-					(reference "SW3")
+					(reference "BOOT")
 					(unit 1)
 				)
@@
 		(dnp no)
 		(fields_autoplaced yes)
-		(property "Reference" "SW2"
+		(property "Reference" "RESET"
 			(at 26.67 29.21 0)
 			(effects
@@
 			)
 		)
-		(property "Value" "SW_Push"
+		(property "Value" "RESET"
 			(at 26.67 31.75 0)
 			(effects
@@
 			(project "PCB"
 				(path "/7d2cf6c2-cd4f-44e4-8c0c-48fa8c8e68c1"
-					(reference "SW2")
+					(reference "RESET")
 					(unit 1)
 				)

Commit message: potato
Parts:
- renumbered BOOT to BOOT1, RESET to RESET1
Changed lines of the file:
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@@
 		(dnp no)
 		(fields_autoplaced yes)
-		(property "Reference" "BOOT"
+		(property "Reference" "BOOT1"
 			(at 154.94 52.07 0)
 			(effects
@@
 			(project "PCB"
 				(path "/7d2cf6c2-cd4f-44e4-8c0c-48fa8c8e68c1"
-					(reference "BOOT")
+					(reference "BOOT1")
 					(unit 1)
 				)
@@
 		(dnp no)
 		(fields_autoplaced yes)
-		(property "Reference" "RESET"
+		(property "Reference" "RESET1"
 			(at 26.67 29.21 0)
 			(effects
@@
 			(project "PCB"
 				(path "/7d2cf6c2-cd4f-44e4-8c0c-48fa8c8e68c1"
-					(reference "RESET")
+					(reference "RESET1")
 					(unit 1)
 				)

Commit message: potato
Parts:
- J1, J2: value Conn_01x07_Pin -> Conn_01x08_Pin
Changed lines of the file:
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@@
 			)
 		)
-		(property "Value" "Conn_01x07_Pin"
+		(property "Value" "Conn_01x08_Pin"
 			(at 170.815 153.67 0)
 			(effects
@@
 			)
 		)
-		(property "Value" "Conn_01x07_Pin"
+		(property "Value" "Conn_01x08_Pin"
 			(at 139.065 154.94 0)
 			(effects
