File: PCB/PCB.kicad_sch (KiCad schematic)
At the start: 39 parts, among them J1 Conn_01x08_Pin, J2 Conn_01x08_Pin, J3 Conn_01x06_Pin, J4 USB_C_Receptacle_USB2.0_14P, J5 Conn_01x03_Pin, U1 RP2040, U2 MCP1700, U3 W25Q128JVS, U4 USBLC6-2SC6, Y1 12MHz

Commit message: potato
Parts:
- R4: value 2.2 -> 2.2k
- R5, R6: value 22k -> 5.1k
Changed lines of the file:
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@@
 			)
 		)
-		(property "Value" "22k"
-			(at 65.786 147.32 90)
+		(property "Value" "5.1k"
+			(at 65.278 145.542 90)
 			(effects
 				(font
@@
 		(on_board yes)
 		(dnp no)
-		(fields_autoplaced yes)
 		(property "Reference" "C11"
 			(at 86.36 146.0562 0)
@@
 		)
 		(property "Value" "10uf"
-			(at 86.36 148.5962 0)
+			(at 77.47 147.32 0)
 			(effects
 				(font
@@
 			)
 		)
-		(property "Value" "2.2"
-			(at 96.52 22.86 90)
+		(property "Value" "2.2k"
+			(at 96.266 21.082 90)
 			(effects
 				(font
@@
 		(dnp no)
 		(property "Reference" "R6"
-			(at 64.008 151.384 90)
+			(at 62.738 151.13 90)
 			(effects
 				(font
@@
 			)
 		)
-		(property "Value" "22k"
-			(at 65.532 149.86 90)
+		(property "Value" "5.1k"
+			(at 64.77 151.638 90)
 			(effects
 				(font
